File: 4-digit/hookup/hookup.sch (KiCad schematic (older format))
At the start: 4 parts, among them J1 Conn_01x05

Commit message: publish
Parts:
- BT1: value 4.5v -> 6v
Connections:
- net at B1.21 (VCC), J1.5 (Pin_5): no longer BT1.1 (+), C1.1
- net at B1.24 (RAW): now also BT1.1 (+), C1.1
- no-connect marks 17 -> 16
Other:
- moved on the sheet: BT1, C1
Changed lines of the file:
@@
 L Device:Battery_Cell BT1
 U 1 1 5DA8A35F
-P 6650 3850
-F 0 "BT1" H 6768 3946 50  0000 L CNN
-F 1 "4.5v" H 6768 3855 50  0000 L CNN
-F 2 "" V 6650 3910 50  0001 C CNN
-F 3 "~" V 6650 3910 50  0001 C CNN
-	1    6650 3850
+P 6450 3550
+F 0 "BT1" H 6568 3646 50  0000 L CNN
+F 1 "6v" H 6568 3555 50  0000 L CNN
+F 2 "" V 6450 3610 50  0001 C CNN
+F 3 "~" V 6450 3610 50  0001 C CNN
+	1    6450 3550
 	1    0    0    -1
 $EndComp
@@
 L Device:C_Small C1
 U 1 1 5DA8ACE6
-P 7150 3750
-F 0 "C1" H 7242 3796 50  0000 L CNN
-F 1 ".1uf" H 7242 3705 50  0000 L CNN
-F 2 "" H 7150 3750 50  0001 C CNN
-F 3 "~" H 7150 3750 50  0001 C CNN
-	1    7150 3750
+P 6950 3450
+F 0 "C1" H 7042 3496 50  0000 L CNN
+F 1 ".1uf" H 7042 3405 50  0000 L CNN
+F 2 "" H 6950 3450 50  0001 C CNN
+F 3 "~" H 6950 3450 50  0001 C CNN
+	1    6950 3450
 	1    0    0    -1
 $EndComp
@@
 	4850 3500 5600 3500
 Wire Wire Line
-	6650 3500 6650 3650
+	6450 3200 6450 3350
 Wire Wire Line
 	5950 4450 5600 4450
 Wire Wire Line
 	5600 4450 5600 3500
-Connection ~ 5600 3500
 Wire Wire Line
-	5600 3500 6650 3500
+	6450 3200 6950 3200
 Wire Wire Line
-	6650 3500 7150 3500
-Wire Wire Line
-	7150 3500 7150 3650
-Connection ~ 6650 3500
+	6950 3200 6950 3350
 $Comp
 L power:GND #PWR?
 U 1 1 5DAB1F24
-P 5300 3700
-F 0 "#PWR?" H 5300 3450 50  0001 C CNN
-F 1 "GND" H 5305 3527 50  0000 C CNN
-F 2 "" H 5300 3700 50  0001 C CNN
-F 3 "" H 5300 3700 50  0001 C CNN
-	1    5300 3700
+P 5800 3700
+F 0 "#PWR?" H 5800 3450 50  0001 C CNN
+F 1 "GND" H 5805 3527 50  0000 C CNN
+F 2 "" H 5800 3700 50  0001 C CNN
+F 3 "" H 5800 3700 50  0001 C CNN
+	1    5800 3700
 	1    0    0    -1
 $EndComp
@@
 L power:GND #PWR?
 U 1 1 5DAB25C8
-P 6650 4150
-F 0 "#PWR?" H 6650 3900 50  0001 C CNN
-F 1 "GND" H 6655 3977 50  0000 C CNN
-F 2 "" H 6650 4150 50  0001 C CNN
-F 3 "" H 6650 4150 50  0001 C CNN
-	1    6650 4150
+P 6450 3850
+F 0 "#PWR?" H 6450 3600 50  0001 C CNN
+F 1 "GND" H 6455 3677 50  0000 C CNN
+F 2 "" H 6450 3850 50  0001 C CNN
+F 3 "" H 6450 3850 50  0001 C CNN
+	1    6450 3850
 	1    0    0    -1
 $EndComp
@@
 L power:GND #PWR?
 U 1 1 5DAB2C6D
-P 7150 4150
-F 0 "#PWR?" H 7150 3900 50  0001 C CNN
-F 1 "GND" H 7155 3977 50  0000 C CNN
-F 2 "" H 7150 4150 50  0001 C CNN
-F 3 "" H 7150 4150 50  0001 C CNN
-	1    7150 4150
+P 6950 3850
+F 0 "#PWR?" H 6950 3600 50  0001 C CNN
+F 1 "GND" H 6955 3677 50  0000 C CNN
+F 2 "" H 6950 3850 50  0001 C CNN
+F 3 "" H 6950 3850 50  0001 C CNN
+	1    6950 3850
 	1    0    0    -1
 $EndComp
@@
 	3250 3500 3250 3750
 Wire Wire Line
-	5300 3700 5300 3300
+	5800 3700 5800 3300
 Wire Wire Line
-	5300 3300 4850 3300
+	5800 3300 4850 3300
 Wire Wire Line
 	5950 4850 5600 4850
@@
 	5600 4850 5600 5000
 Wire Wire Line
-	6650 4150 6650 3950
+	6450 3850 6450 3650
 Wire Wire Line
-	7150 3850 7150 4150
+	6950 3550 6950 3850
 NoConn ~ 3950 3200
 NoConn ~ 3950 3300
@@
 NoConn ~ 3950 4100
 NoConn ~ 3950 4200
-NoConn ~ 4850 3200
 NoConn ~ 4850 3400
 NoConn ~ 4850 3600
@@
 NoConn ~ 4850 4100
 NoConn ~ 4850 4300
+Wire Wire Line
+	6450 3200 4850 3200
+Connection ~ 6450 3200
 $EndSCHEMATC
